File: Schematics/BLDC_driver/BLDC_driver.kicad_sch (KiCad schematic)
At the start: 45 parts, among them J1 DA15_Plug_MountingHoles, J2 Conn_01x02_Pin, J3 Conn_01x07_Pin, J4 USB_B_Micro, J5 DE9_Receptacle_MountingHoles, J7 Conn_01x05_Pin, Q1 2SC4213, Q2 2SC4213, SW1 SW_MEC_5G, SW2 SW_MEC_5G, SW3 SW_MEC_5G, SW4 SW_MEC_5G, U1 TS912, U2 LM2675M-5, U3 CH340C, U4 ESP32-WROOM-32D, U5 MAX3232, U6 AMS1117-3.3, U7 TS912, U8 AMS1117-3.3

Commit message: Further Schematic Progress
Added some components, assigned most of the footprints, one more commit. All basic functionalities considered in the schematic.
Parts:
- removed DISP1: ~, symbol Modules:1.3''_OLED_DISPLAY
- removed J2: Conn_01x02_Pin, Connector_PinHeader_2.54mm:PinHeader_1x02_P2.54mm_Vertical, symbol Connector:Conn_01x02_Pin
- removed J7: Conn_01x05_Pin, symbol Connector:Conn_01x05_Pin
- removed Q1, Q2: 2SC4213, Package_TO_SOT_SMD:SOT-323_SC-70, symbol Transistor_BJT:2SC4213
- removed R1, R2: 10k, symbol Device:R
- removed U1, U7: TS912, symbol Amplifier_Operational:TS912
- added C11: 100n, Capacitor_SMD:C_0402_1005Metric_Pad0.74x0.62mm_HandSolder, symbol Device:C_Small
- added C16, C17: 0.1u, symbol Device:C
- added H1, H2, H3, H4, H5, H6, H7, H8: MountingHole, MountingHole:MountingHole_3.2mm_M3_Pad_Via, symbol Mechanical:MountingHole_Pad
- added J2: Display connectors, Connector_PinHeader_2.54mm:PinHeader_1x04_P2.54mm_Vertical, symbol Connector:Conn_01x04_Pin
- added J6: Programmer IO, Connector_PinHeader_2.54mm:PinHeader_1x06_P2.54mm_Vertical, symbol Connector:Conn_01x07_Pin
- added J7: Conn_02x08_Counter_Clockwise, Connector_PinHeader_2.54mm:PinHeader_2x08_P2.54mm_Vertical, symbol Connector_Generic:Conn_02x08_Counter_Clockwise
- added Q1: UMH3N, Package_TO_SOT_SMD:SOT-363_SC-70-6, symbol Transistor_BJT:UMH3N
- added R1: 10K, Resistor_SMD:R_0402_1005Metric_Pad0.72x0.64mm_HandSolder, symbol Device:R_Small
- added R10, R11, R6, R8, R9: 10k, Resistor_SMD:R_0402_1005Metric_Pad0.72x0.64mm_HandSolder, symbol Device:R_Small
- added R2: 7k5, Resistor_SMD:R_0402_1005Metric_Pad0.72x0.64mm_HandSolder, symbol Device:R_Small
- added R7: 1k6, Resistor_SMD:R_0402_1005Metric_Pad0.72x0.64mm_HandSolder, symbol Device:R_Small
- added SW5: En_switch, symbol Switch:SW_MEC_5G
- added U1: ICL7660, Package_SO:PowerIntegrations_SO-8, symbol Regulator_SwitchedCapacitor:ICL7660
- added U7: LM358, Package_DIP:DIP-8_W7.62mm, symbol Amplifier_Operational:LM358
- C1: value 10u -> 22u
- J1: footprint Connector_Dsub:DSUB-15_Female_Horizontal_P2.77x2.84mm_EdgePinOffset4.94mm_Housed_MountingHolesOffset7.48mm -> Connector_Dsub:DSUB-15_Female_Vertical_P2.77x2.84mm_MountingHoles
- J4: footprint (none) -> Connector_USB:USB_Mini-B_Wuerth_65100516121_Horizontal
- J5: footprint (none) -> Connector_Dsub:DSUB-9_Female_Vertical_P2.77x2.84mm_MountingHoles
- L1: renamed from 47u; value L -> 47u
- U4: footprint RF_Module:ESP32-WROOM-32D -> esp32:ESP32-WROOM-32E
- renumbered 150u/35v to 150u/35v1
Connections:
- net +3.3V: now also J2.1 (Pin_1), J6.6 (Pin_6), R1.1
- net +5V: now also J6.5 (Pin_5), U1.8 (V+), U7.8 (V+)
- net CTRL: now also R11.2, U7.7
- net DAC1: now also R8.1
- net DAC2: now also R9.1
- net DTR: now also Q1.2 (B1), Q1.3 (C2)
- net EN: now also C11.1, J6.3 (Pin_3), R1.2, SW5.3 (B), SW5.4 (B)
- net EN USB: now also Q1.6 (C1)
- net GND: now also U4.1 (GND), U4.15 (GND), U4.38 (GND), U4.39 (GND), C11.2, C17.1, H1.1, H2.1, H3.1, H4.1, J2.2 (Pin_2), J6.7 (Pin_7), R7.2, SW5.1 (A), SW5.2 (A), U1.3 (GND), U7.3 (+), U7.5 (+); no longer C13.2, C15.2, C8.2, J3.7 (Pin_7), J4.4 (ID), J4.5 (GND), J4.6 (Shield), R5.2, U3.1 (GND), U8.1 (GND)
- net GPIO0: now also J6.4 (Pin_4); no longer J3.4 (Pin_4)
- net GPIO0 USB: now also J3.4 (Pin_4), Q1.4 (E2)
- net RPM: now also R6.1
- net RTS: now also Q1.1 (E1), Q1.5 (B2)
- net SCL: now also J2.3 (Pin_3)
- net SDA: now also J2.4 (Pin_4)
- net U0RX: now also J6.1 (Pin_1)
- net U0TX: now also J6.2 (Pin_2); no longer J3.2 (Pin_2)
- net U0TX USB: now also J3.2 (Pin_2)
- net O1 renamed RPM DIVIDED
- net RPM DIVIDED: now also R6.2, R7.1
- new net: R10.2, R11.1, U7.6 (-)
- new net: R10.1, R2.2, U7.1
- new net: R2.1, R8.2, R9.2, U7.2 (-)
- new net: C16.1, U1.2 (CAP+)
- new net: C16.2, U1.4 (CAP-)
- new net -5V: C17.2, U1.5 (VOUT), U7.4 (V-)
- new net GND1: C13.2, C15.2, C8.2, H5.1, H6.1, H7.1, H8.1, J3.7 (Pin_7), J4.4 (ID), J4.5 (GND), J4.6 (Shield), R5.2, U3.1 (GND), U8.1 (GND)
- no-connect marks 25 -> 28
Other:
- note added: "Power"
- moved on the sheet: 150u/35v1, C1, C10, C12, C14, C2, C3, C4, C5, C6, C7, C9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

Commit message: Finished design
Generated gerber files, upgraded to KiCAD 8.0.7 this is final design (hopefully)
Parts:
- removed C12: 10n+ ceramic, symbol Device:C
- removed D1: 1N58xx, Diode_THT:D_DO-201AD_P15.24mm_Horizontal, symbol Diode:1N5822
- removed J7: Conn_02x08_Counter_Clockwise, Connector_PinHeader_2.54mm:PinHeader_2x08_P2.54mm_Vertical, symbol Connector_Generic:Conn_02x08_Counter_Clockwise
- removed Q1: UMH3N, Package_TO_SOT_SMD:SOT-363_SC-70-6, symbol Transistor_BJT:UMH3N
- removed SW1, SW2, SW3, SW4: SW_MEC_5G, symbol Switch:SW_MEC_5G
- removed SW5: En_switch, symbol Switch:SW_MEC_5G
- removed U2: LM2675M-5, Package_SO:SOIC-8_3.9x4.9mm_P1.27mm, symbol Regulator_Switching:LM2675M-5
- removed U4: ESP32-WROOM-32D, esp32:ESP32-WROOM-32E, symbol RF_Module:ESP32-WROOM-32D
- added C6: 22u, Capacitor_SMD:C_0805_2012Metric_Pad1.18x1.45mm_HandSolder, symbol Device:C
- added D2: B320, Diode_SMD:D_SMC_Handsoldering, symbol Diode:B320
- added J4: unused pins, Connector_PinHeader_2.54mm:PinHeader_1x12_P2.54mm_Vertical, symbol Connector_Generic:Conn_02x06_Counter_Clockwise
- added Q1, Q2, Q3: 2N7002, Package_TO_SOT_SMD:SOT-23, symbol Transistor_FET:2N7002
- added R10: 100, Resistor_SMD:R_0402_1005Metric_Pad0.72x0.64mm_HandSolder, symbol Device:R_Small
- added R12: 10k, Resistor_SMD:R_0402_1005Metric_Pad0.72x0.64mm_HandSolder, symbol Device:R_Small
- added R14, R15: 10k, Resistor_SMD:R_0402_1005Metric_Pad0.72x0.64mm_HandSolder, symbol Device:R
- added R16, R17: 3k3, Resistor_SMD:R_0402_1005Metric_Pad0.72x0.64mm_HandSolder, symbol Device:R_Small
- added SW1, SW2, SW3, SW4, SW5: SW_Push, PCM_Espressif:SW_Push_1P1T_NO_CK_KSC6xxJ22, symbol Switch:SW_Push
- added U1: ESP32-WROOM-E, PCM_Espressif:ESP32-WROOM-32E, symbol PCM_Espressif:ESP32-WROOM-E
- added U2: LM2596S-5, Package_TO_SOT_SMD:TO-263-5_TabPin3, symbol Regulator_Switching:LM2596S-5
- C1: footprint (none) -> Capacitor_SMD:C_0805_2012Metric_Pad1.18x1.45mm_HandSolder
- C10: renamed from C11; value 100n -> 0.1u; footprint Capacitor_SMD:C_0402_1005Metric_Pad0.74x0.62mm_HandSolder -> Capacitor_SMD:C_0603_1608Metric_Pad1.08x0.95mm_HandSolder
- C11: renamed from 150u/35v1; value C -> 220u/35v; footprint (none) -> Capacitor_THT:CP_Radial_D8.0mm_P3.50mm
- C12: renamed from C3; footprint (none) -> Capacitor_SMD:C_0603_1608Metric_Pad1.08x0.95mm_HandSolder
- C13: renamed from C5; footprint (none) -> Capacitor_SMD:C_0603_1608Metric_Pad1.08x0.95mm_HandSolder
- C14: renamed from C4; footprint (none) -> Capacitor_SMD:C_0603_1608Metric_Pad1.08x0.95mm_HandSolder
- C15: renamed from C6; footprint (none) -> Capacitor_SMD:C_0603_1608Metric_Pad1.08x0.95mm_HandSolder
- C16: renamed from C7; footprint (none) -> Capacitor_SMD:C_0603_1608Metric_Pad1.08x0.95mm_HandSolder
- C17: renamed from C13; footprint (none) -> Capacitor_SMD:C_0805_2012Metric_Pad1.18x1.45mm_HandSolder
- C18: renamed from C15; footprint (none) -> Capacitor_SMD:C_0805_2012Metric_Pad1.18x1.45mm_HandSolder
- C19: renamed from C8; footprint (none) -> Capacitor_SMD:C_0603_1608Metric_Pad1.08x0.95mm_HandSolder
- C2: footprint (none) -> Capacitor_SMD:C_0603_1608Metric_Pad1.08x0.95mm_HandSolder
- C3: renamed from C17; footprint (none) -> Capacitor_SMD:C_0603_1608Metric_Pad1.08x0.95mm_HandSolder
- C4: renamed from C9; footprint (none) -> Capacitor_SMD:C_0805_2012Metric_Pad1.18x1.45mm_HandSolder
- C5: renamed from C10; footprint (none) -> Capacitor_SMD:C_0805_2012Metric_Pad1.18x1.45mm_HandSolder
- C8: renamed from C16; footprint (none) -> Capacitor_SMD:C_0603_1608Metric_Pad1.08x0.95mm_HandSolder
- C9: renamed from C14; value 150u/35v -> 220u/35v; footprint (none) -> Capacitor_THT:CP_Radial_D8.0mm_P3.50mm
- D1: renamed from D2; footprint (none) -> Diode_SMD:D_0603_1608Metric_Pad1.05x0.95mm_HandSolder
- D3: footprint (none) -> Diode_SMD:D_0603_1608Metric_Pad1.05x0.95mm_HandSolder
- J3: renamed from J6; footprint Connector_PinHeader_2.54mm:PinHeader_1x06_P2.54mm_Vertical -> Connector_PinHeader_2.54mm:PinHeader_1x07_P2.54mm_Vertical
- J6: renamed from J3; footprint (none) -> Connector_PinHeader_2.54mm:PinHeader_1x07_P2.54mm_Vertical
- L1: value 47u -> 33u; footprint (none) -> Inductor_SMD:L_Coilcraft_MSS1278T-XXX
- R1: renamed from R6; footprint Resistor_SMD:R_0402_1005Metric_Pad0.72x0.64mm_HandSolder -> Resistor_THT:R_Axial_DIN0207_L6.3mm_D2.5mm_P10.16mm_Horizontal
- R11: renamed from R4; footprint (none) -> Resistor_SMD:R_0402_1005Metric_Pad0.72x0.64mm_HandSolder
- R13: renamed from R5; footprint (none) -> Resistor_SMD:R_0402_1005Metric_Pad0.72x0.64mm_HandSolder
- R2: renamed from R1; value 10K -> 10k
- R3: renamed from R7; footprint Resistor_SMD:R_0402_1005Metric_Pad0.72x0.64mm_HandSolder -> Resistor_THT:R_Axial_DIN0207_L6.3mm_D2.5mm_P10.16mm_Horizontal
- R4: renamed from R3; footprint (none) -> Resistor_SMD:R_0402_1005Metric_Pad0.72x0.64mm_HandSolder
- U3: renamed from U6; footprint Package_TO_SOT_SMD:SOT-223-3_TabPin2 -> Package_TO_SOT_SMD:SOT-223
- U6: renamed from U5; footprint Package_SO:SOIC-16_3.9x9.9mm_P1.27mm -> Package_SO:SOP-16_3.9x9.9mm_P1.27mm
- U7: renamed from U8; footprint Package_TO_SOT_SMD:SOT-223-3_TabPin2 -> Package_TO_SOT_SMD:SOT-223
- renumbered J4 to J7, R2 to R5, R11 to R6, R8 to R7, R10 to R8, U7 to U4, U1 to U5, U3 to U8
Connections:
- net +24V: now also U2.1 (VIN)
- net +3.3V: now also R16.1, R17.1, U1.2 (3V3)
- net +5V: now also R10.1, U2.4 (FB)
- net CTRL: now also J4.6 (Pin_6)
- net DAC1: now also U1.10 (DAC_1/ADC2_CH8/GPIO25)
- net DAC2: now also U1.11 (DAC_2/ADC2_CH9/GPIO26)
- net DIR: now also Q1.3 (D), R10.2
- net DTR: now also Q3.2 (S), R14.2
- net EN: now also SW1.2, U1.3 (EN/CHIP_PU)
- net EN USB: now also Q2.3 (D)
- net GND: now also C6.2, D2.2 (A), Q1.2 (S), SW1.1, U1.1 (GND), U1.15 (GND), U1.38 (GND), U1.39 (GND_THERMAL), U2.3 (GND), U2.5 (~{ON}/OFF)
- net GPIO0: now also U1.25 (GPIO0/BOOT/ADC2_CH1)
- net GPIO0 USB: now also Q3.3 (D)
- net RPM DIVIDED: now also C6.1, U1.6 (GPIO34/ADC1_CH6)
- net RTS: now also Q2.2 (S), R15.2
- net SCL: now also R16.2, U1.36 (GPIO22)
- net SDA: now also R17.2, U1.33 (GPIO21)
- net SW1: now also SW2.1, U1.30 (GPIO18)
- net SW2: now also SW3.1, U1.37 (GPIO23)
- net SW3: now also SW4.1, U1.31 (GPIO19)
- net SW4: now also SW5.1, U1.29 (GPIO5)
- net U0RX: now also U1.34 (U0RXD/GPIO3)
- net U0TX: now also U1.35 (U0TXD/GPIO1)
- net U2RX: now also U1.27 (GPIO16)
- net U2TX: now also U1.28 (GPIO17)
- net at L1.1: now also D2.1 (K), U2.2 (OUT)
- net at R11.1: now also SW2.2, SW3.2, SW4.2, SW5.2
- net D-: now reaches J7.2 (D-), U8.6 (UD-)
- net D+: now reaches J7.3 (D+), U8.5 (UD+)
- new net: Q3.1 (G), R15.1
- new net: Q2.1 (G), R14.1
- new net: Q1.1 (G), R12.2
- new net DIR control: R12.1, U1.12 (ADC2_CH7/GPIO27)
- new net IO12: J4.10 (Pin_10), U1.14 (MTDI/GPIO12/ADC2_CH5)
- new net IO13: J4.9 (Pin_9), U1.16 (MTCK/GPIO13/ADC2_CH4)
- new net IO14: J4.8 (Pin_8), U1.13 (MTMS/GPIO14/ADC2_CH6)
- new net IO15: J4.7 (Pin_7), U1.23 (MTDO/GPIO15/ADC2_CH3)
- new net IO2: J4.11 (Pin_11), U1.24 (ADC2_CH2/GPIO2)
- new net IO32: J4.1 (Pin_1), U1.8 (32K_XP/GPIO32/ADC1_CH4)
- new net IO33: J4.2 (Pin_2), U1.9 (32K_XN/GPIO33/ADC1_CH5)
- new net IO35: J4.3 (Pin_3), U1.7 (GPIO35/ADC1_CH7)
- new net IO36: J4.4 (Pin_4), U1.4 (SENSOR_VP/GPIO36/ADC1_CH0)
- new net IO39: J4.5 (Pin_5), U1.5 (SENSOR_VN/GPIO39/ADC1_CH3)
- new net IO4: J4.12 (Pin_12), U1.26 (ADC2_CH0/GPIO4)
- no-connect marks 28 -> 27
Other:
- moved on the sheet: C1, C10, C11, C12, C13, C14, C15, C16, C2, C9, H1, H2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
