File: Schematics/BLDC_driver/BLDC_driver.kicad_sch (KiCad schematic)
At the start: 70 parts, among them J1 DA15_Plug_MountingHoles, J2 Display connectors, J3 Programmer IO, J4 unused pins, J5 DE9_Receptacle_MountingHoles, J6 Conn_01x07_Pin, J7 USB_B_Micro, Q1 2N7002, Q2 2N7002, Q3 2N7002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

Commit message: Skończono opis hardware
Napisano całą część hardwere'ową pracy, do tego poprawiono element z wzmacniaczem na schemacie, żeby tylko jeszcze przyszedł na czas.
Parts:
- D1: value RED -> led
- R5: value 7k5 -> 75k
- R6, R7, R9: value 10k -> 100k
- U4: value LM358 -> LMC6482
Other:
- moved on the sheet: J2, J3, J4, R16, R17

Commit message: Testing board code complete, document had first review
Parts:
- removed C6: 22u, Capacitor_SMD:C_0805_2012Metric_Pad1.18x1.45mm_HandSolder, symbol Device:C
- R8: value 10k -> 100k
Other:
- moved on the sheet: Q1, R10, R11, R12, R6, SW2, SW3, SW4, SW5
